File: expt_01_FaceFollowing/KiCad/01_FaceFollowing/01_FaceFollowing.kicad_sch (KiCad schematic)
At the start: 1 part, among them U1 XIAO ESP32C3

Commit message: prelim schematic
Parts:
- added C1, C2: 1 uF, symbol Device:C_Small_US
- added Hallowing_U2: ~, symbol mdoLibrary:Hallowing_M4
- added R1, R2: 5K, symbol Device:R_Small_US
- added U2: Vision-AI V2 Connector, symbol mdoLibrary:VisionAIv2_cnctr
Connections:
- new net: C2.1, Hallowing_U2. (A5), R2.2
- new net: U1. (D07), U2. (TXD) (x6)
- new net: C1.1, Hallowing_U2. (A5), R1.2
- new net: R2.1, U1. (D07)
- new net: R1.1, U1. (D07)
- new net GND: C1.2, C2.2
Other:
- note added: "GND and +5V via USB"
- company: (none) -> Self: https://github.com/Mark-MDO47
- title: (none) -> https://github.com/Mark-MDO47/expts_grove_vision_ai_v2
- moved on the sheet: U1

Commit message: expt_01a_Analog
Connections:
- net at U2. (TXD): now also U1. (D07)
- net at U1. (D07): no longer U2. (TXD)
- net at Hallowing_U2. (A5): now also C1.1, R1.2
- new net: U1. (D07), U2. (TXD) (x5)
- now unconnected: U1. (D07), U1. (D07), U1. (D07), U1. (D07), U1. (D07)
Other:
- note added: "+"
Changed lines of the file:
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@@
 	(title_block
 		(title "https://github.com/Mark-MDO47/expts_grove_vision_ai_v2")
-		(date "2025-10-04")
+		(date "2025-10-10")
 		(company "Self: https://github.com/Mark-MDO47")
 	)
@@
 				(bold yes)
 			)
+		)
+	)
+	(text "+"
+		(exclude_from_sim no)
+		(at 154.94 126.238 0)
+		(effects
+			(font
+				(size 2 2)
+				(thickness 0.4)
+				(bold yes)
+			)
+		)
+	)
+	(text "+"
+		(exclude_from_sim no)
+		(at 167.64 126.238 0)
+		(effects
+			(font
+				(size 2 2)
+				(thickness 0.4)
+				(bold yes)
+			)
